Commit message: tested gazebo sim control

File: robotis_mini_ros/robotis_mini_description/urdf/servo.urdf.xacro (robot description, xacro)
@@ -4,16 +4,16 @@
        xmlns:interface="http://playerstage.sourceforge.net/gazebo/xmlschema/#interface"
        xmlns:xacro="http://ros.org/wiki/xacro">
-  <property name="M_PI" value="3.1415926535897931" />
-  <property name="XL320_MAX_TORQUE" value="0.39" />
-  <property name="XL320_MAX_VELOCITY" value="${114 * 2*M_PI / 60}" />
-  <property name="XL320_DAMPING" value="0.7" />
+  <xacro:property name="M_PI" value="3.1415926535897931" />
+  <xacro:property name="XL320_MAX_TORQUE" value="0.39" />
+  <xacro:property name="XL320_MAX_VELOCITY" value="${114 * 2*M_PI / 60}" />
+  <xacro:property name="XL320_DAMPING" value="0.7" />
   <xacro:macro name="robotis_mini_transmission" params="name">
     <transmission name="${name}_tran">
       <type>transmission_interface/SimpleTransmission</type>
       <joint name="${name}_joint">
-        <hardwareInterface>EffortJointInterface</hardwareInterface>
+        <hardwareInterface>hardware_interface/EffortJointInterface</hardwareInterface>
       </joint>
       <actuator name="${name}_motor">
-        <hardwareInterface>EffortJointInterface</hardwareInterface>
+        <hardwareInterface>hardware_interface/EffortJointInterface</hardwareInterface>
         <mechanicalReduction>1</mechanicalReduction>
       </actuator>
