Commit message: replaced body with upgrade kit

File: robotis_mini_ros/robotis_mini_description/urdf/arm.urdf.xacro (robot description, xacro)
@@ -3,5 +3,5 @@
   <xacro:macro name="robotis_mini_arm" params="side parent reflect">
     <xacro:robotis_mini_servo_fixed name="${side}_shoulder" parent="${parent}"
-        xyz="0 -0.024 0" rpy="${(1-reflect)*M_PI/2} 0 ${(1+reflect)*M_PI/2}" initial_rotation="0" reflect="${reflect}"/>
+        xyz="0 0 0" rpy="${(1-reflect)*M_PI/2} 0 ${(1+reflect)*M_PI/2}" initial_rotation="0" reflect="${reflect}"/>
     <xacro:robotis_mini_dmfb03 name="${side}_biceps_anchor" parent="${side}_shoulder_link"
         xyz="${reflect*0.012} 0 0.033" rpy="${M_PI/2} 0 ${reflect*-M_PI/2}" />

File: robotis_mini_ros/robotis_mini_description/urdf/body.urdf.xacro (robot description, xacro)
@@ -26,3 +26,7 @@
         xyz="-0.024 -0.006 -0.033" rpy="0 0 0" />
   </xacro:macro>
+  <xacro:macro name="robotis_mini_body2" params="parent">
+    <xacro:robotis_mini_upgrade_body name="robotis_mini_upgrade" parent="${parent}"
+        xyz="0 0 0" rpy="-${M_PI/2} 0 0" />
+  </xacro:macro>
 </robot>

File: robotis_mini_ros/robotis_mini_description/urdf/common.urdf.xacro (robot description, xacro)
@@ -59,5 +59,5 @@
       <mu1>10000</mu1>
       <mu2>10000</mu2>
-      <kp>100.0</kp>
+      <kp>10000.0</kp>
       <kd>100.0</kd>
       <minDepth>0.001</minDepth>
@@ -65,4 +65,74 @@
     </gazebo>
   </xacro:macro>
+  <xacro:macro name="robotis_mini_upgrade_body" params="name parent xyz rpy">
+    <joint name="${name}_joint" type="fixed">
+      <origin xyz="${xyz}" rpy="${rpy}" />
+      <parent link="${parent}"/>
+      <child link="${name}_link"/>
+    </joint>
+    <link name="${name}_link">
+      <inertial>
+        <origin
+          xyz="-0.0091918 -0.00047008 -0.016078"
+          rpy="0 0 0" />
+        <mass
+          value="0.2437" />
+        <inertia
+          ixx="9.5353E-05"
+          ixy="-3.5005E-08"
+          ixz="-9.1096E-06"
+          iyy="6.6853E-05"
+          iyz="7.5168E-07"
+          izz="9.5174E-05" />
+      </inertial>
+      <visual>
+        <origin
+          xyz="0 0 0"
+          rpy="0 0 0" />
+        <geometry>
+          <mesh
+            filename="package://robotis_mini/meshes/Body.STL" />
+        </geometry>
+        <material
+          name="">
+          <color
+            rgba="0.75294 0.75294 0.75294 1" />
+        </material>
+      </visual>
+      <collision>
+        <origin
+          xyz="0 0 0"
+          rpy="0 0 0" />
+        <geometry>
+          <mesh
+            filename="package://robotis_mini/meshes/Body.STL" />
+        </geometry>
+      </collision>
+    </link>
+    <link name="left_arm_socket_link" />
+    <joint name="left_arm_socket_joint" type="fixed">
+      <parent link="${name}_link"/>
+      <child link="left_arm_socket_link"/>
+      <origin xyz="0 0 0.038998" rpy="0 0 -1.5708" />
+    </joint>
+    <link name="right_arm_socket_link" />
+    <joint name="right_arm_socket_joint" type="fixed">
+      <parent link="${name}_link"/>
+      <child link="right_arm_socket_link"/>
+      <origin xyz="0 0 -0.038998" rpy="0 0 -1.5708" />
+    </joint>
+    <link name="left_leg_socket_link" />
+    <joint name="left_leg_socket_joint" type="fixed">
+      <parent link="${name}_link"/>
+      <child link="left_leg_socket_link"/>
+      <origin xyz="0 0.072 0.024" rpy="1.5633 -1.5708 1.5708" />
+    </joint>
+    <link name="right_leg_socket_link" />
+    <joint name="right_leg_socket_joint" type="fixed">
+      <parent link="${name}_link"/>
+      <child link="right_leg_socket_link"/>
+      <origin xyz="0 0.072 -0.024" rpy="1.5708 -1.5708 1.5708" />
+    </joint>
+  </xacro:macro>
   <xacro:macro name="robotis_mini_dmfb01" params="name parent xyz rpy">
     <joint name="${name}_joint" type="fixed">

File: robotis_mini_ros/robotis_mini_description/urdf/leg.urdf.xacro (robot description, xacro)
@@ -6,5 +6,5 @@
   <xacro:macro name="robotis_mini_leg" params="side parent reflect">
     <xacro:robotis_mini_servo_fixed name="${side}_hip" parent="${parent}"
-        xyz="0 -0.024 0" rpy="0 0 ${M_PI}" initial_rotation="0" reflect="${-reflect}"/>
+        xyz="0 0 0" rpy="0 0 ${M_PI}" initial_rotation="0" reflect="${-reflect}"/>
     <xacro:robotis_mini_spd7v4 name="${side}_groin" parent="${side}_hip_link"
         xyz="0 0 0.0165" rpy="${-M_PI/2} 0 ${-M_PI/2}" />

File: robotis_mini_ros/robotis_mini_description/urdf/robotis_mini.urdf.xacro (robot description, xacro)
@@ -14,9 +14,9 @@
   <xacro:include filename="$(find robotis_mini_description)/urdf/leg.urdf.xacro" />
   <xacro:robotis_mini_base name="base"/>
-  <xacro:robotis_mini_body parent="base_link" />
-  <xacro:robotis_mini_arm side="l" reflect="1" parent="l_shoulder_anchor_link" />
-  <xacro:robotis_mini_arm side="r" reflect="-1" parent="r_shoulder_anchor_link" />
-  <xacro:robotis_mini_leg side="l" reflect="1" parent="l_hip_anchor_link" />
-  <xacro:robotis_mini_leg side="r" reflect="-1" parent="r_hip_anchor_link" />
+  <xacro:robotis_mini_body2 parent="base_link" />
+  <xacro:robotis_mini_arm side="l" reflect="1" parent="left_arm_socket_link" />
+  <xacro:robotis_mini_arm side="r" reflect="-1" parent="right_arm_socket_link" />
+  <xacro:robotis_mini_leg side="l" reflect="1" parent="left_leg_socket_link" />
+  <xacro:robotis_mini_leg side="r" reflect="-1" parent="right_leg_socket_link" />
   <gazebo>
     <plugin name="gazebo_ros_control" filename="libgazebo_ros_control.so">
